File: DIY Arduboy Flash module KiCad Files/diy_ardubo_flash_module.kicad_sch (KiCad schematic)
At the start: 21 parts, among them J1 Conn_02x01, J2 Conn_01x07_Pin, J3 Conn_02x03_Odd_Even, J4 Conn_01x06_Pin, J5 Conn_01x01_Pin, Q1 BC557, SW1 SW_Push, SW2 SW_Push, SW3 SW_Push, SW4 SW_Push, SW5 SW_Push, SW6 SW_Push, SW7 SW_Push, SW8 SW_SPDT, U1 ProMicro

Commit message: Updated Schematics
Fixed ground pin issue with switch
Parts:
- removed J1: Conn_02x01, Connector_PinHeader_2.54mm:PinHeader_2x01_P2.54mm_Vertical, symbol Connector_Generic:Conn_02x01
- added J1, J6, J7: Conn_01x02_Pin, Connector_PinHeader_2.54mm:PinHeader_1x02_P2.54mm_Vertical, symbol Connector:Conn_01x02_Pin
Connections:
- net at SW8.2 (B): now also J6.1 (Pin_1)
- net at U1.24 (RAW): now also J7.1 (Pin_1)
- net at C1.2, J2.1 (GND), J4.3 (Pin_3)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: now also J7.2 (Pin_2); no longer SW8.3 (C)
- net at SW8.1 (A): now also J1.1 (Pin_1)
- new net: J1.2 (Pin_2), J6.2 (Pin_2)
